Commit message: update setup

File: race_float_description/urdf/base.urdf (robot description, URDF)
Before this commit: robot float_rise, 6 links, 5 joints
Links:
- removed link gps
- removed link nose_tip_link
- added link light
- added link tag1
- added link tag2
Joints:
- removed joint gps_joint
- added joint light_joint: type fixed, parent base_link, child light, origin xyz=0.075 0.0 0.635 rpy=3.1415926 0.0 0.0
- added joint tag1_joint: type fixed, parent base_link, child tag1, origin xyz=0.075 0.0 0.635 rpy=3.1415926 0.0 0.0
- added joint tag2_joint: type fixed, parent base_link, child tag2, origin xyz=0.075 0.0 0.635 rpy=3.1415926 0.0 0.0
- joint base_link: child nose_tip_link -> (none)
- joint imu_joint: origin xyz=-0.2 -0.07 0.0 rpy=0.0 0.0 0.0 -> xyz=0.0 0.0 0.0 rpy=0.0 0.0 0.0

Commit message: updated

File: race_float_description/urdf/base.urdf (robot description, URDF)
Before this commit: robot race_float, 7 links, 7 joints
Joints:
- joint cg_joint: origin xyz=0.0 0.0 0.0 rpy=3.1415926 0.0 0.0 -> xyz=0.0 0.0 0.0 rpy=0.0 0.0 0.0
- joint light_joint: origin xyz=0.075 0.0 0.635 rpy=3.1415926 0.0 0.0 -> xyz=-0.02 0.03 0.157 rpy=0.0 0.0 0.0
- joint pressure_joint: origin xyz=0.00 0.0 -0.02 rpy=3.1415926 0.0 0.0 -> xyz=0.00 0.0 -0.02 rpy=0.0 0.0 0.0
- joint tag1_joint: origin xyz=0.075 0.0 0.635 rpy=3.1415926 0.0 0.0 -> xyz=0.0 0.0 0.122 rpy=0.0 0.0 0.0
- joint tag2_joint: origin xyz=0.075 0.0 0.635 rpy=3.1415926 0.0 0.0 -> xyz=0.0 0.0 0.20 rpy=0.0 0.0 0.0

Commit message: set up robot localization

File: race_float_description/urdf/base.urdf (robot description, URDF)
Before this commit: robot race_float, 7 links, 7 joints
Links:
- removed link tag1
- removed link tag2
- added link gps
- added link tag17
- added link tag25
Joints:
- removed joint base_link
- added joint gps_joint: type fixed, parent base_link, child gps, origin xyz=0.0 0.0 0.0 rpy=0.0 0.0 0.0
- joint light_joint: origin xyz=-0.02 0.03 0.157 rpy=0.0 0.0 0.0 -> xyz=-0.02 0.03 1.57 rpy=-90.0 0.0 180.0
- joint tag1_joint: child tag1 -> tag25; origin xyz=0.0 0.0 0.122 rpy=0.0 0.0 0.0 -> xyz=0.0 0.0 1.22 rpy=0.0 -90.0 -90.0
- joint tag2_joint: child tag2 -> tag17; origin xyz=0.0 0.0 0.20 rpy=0.0 0.0 0.0 -> xyz=0.0 0.0 2.0 rpy=-90.0 90.0 0.0
