Commit message: race station update

File: race_float_description/urdf/base.urdf (robot description, URDF)
Before this commit: robot race_float, 8 links, 7 joints
Links:
- removed link light
- removed link tag17
- removed link tag25
- added link apriltag25h9_02
- added link apriltag25h9_13
- added link apriltag25h9_17
- added link apriltag25h9_25
- added link apriltag36h11_009
- added link apriltag36h11_022
- added link dock_point
- added link imu_sf
- added link nose_tip_link
Joints:
- removed joint light_joint
- removed joint tag1_joint
- removed joint tag2_joint
- added joint apriltag25h9_02_joint: type fixed, parent base_link, child apriltag25h9_02, origin xyz=0.0 0.33 0.17 rpy=0.0 1.5707963 0.0
- added joint apriltag25h9_13_joint: type fixed, parent base_link, child apriltag25h9_13, origin xyz=-0.65 0.68 0.17 rpy=1.5707963 1.5707963 3.1415926
- added joint apriltag25h9_17_joint: type fixed, parent base_link, child apriltag25h9_17, origin xyz=-1.22 0.33 0.17 rpy=0.0 1.5707963 3.1415926
- added joint apriltag25h9_25_joint: type fixed, parent base_link, child apriltag25h9_25, origin xyz=-0.65 -0.03 0.17 rpy=1.5707963 1.5707963 0.0
- added joint apriltag36h11_009_joint: type fixed, parent base_link, child apriltag36h11_009, origin xyz=-0.42 0.12 0.0 rpy=0.0 3.1415926 3.1415926
- added joint apriltag36h11_022_joint: type fixed, parent base_link, child apriltag36h11_022, origin xyz=-0.42 0.52 0.0 rpy=0.0 3.1415926 3.1415926
- added joint base_link: type fixed, parent base_link, child nose_tip_link, origin xyz=0.0 0.0 0.0 rpy=0.0 0.0 0.0
- added joint dock_point_joint: type fixed, parent base_link, child dock_point, origin xyz=-0.415 0.33 -0.05 rpy=0.0 0.0 0.0
- added joint imu__sf_joint: type fixed, parent base_link, child imu_sf, origin xyz=0.0 0.0 0.0 rpy=0.0 0.0 0.0
- joint cg_joint: origin xyz=0.0 0.0 0.0 rpy=0.0 0.0 0.0 -> xyz=0.0 0.0 0.0 rpy=3.1415926 0.0 0.0
- joint pressure_joint: origin xyz=0.00 0.0 -0.02 rpy=0.0 0.0 0.0 -> xyz=0.0 0.0 0.0 rpy=0.0 0.0 0.0
